Commit message: 验证匹配端；镭射和仿真实测22.04 pcl做原来的帧间匹配慢几十倍；仿真可视化优化

File: src/genshin_simulation/urdf/HDL-32E.xacro (robot description, xacro)
@@ -2,5 +2,5 @@
 <robot xmlns:xacro="http://www.ros.org/wiki/xacro" name="HDL-32E">
   <xacro:property name="M_PI" value="3.1415926535897931" />
-  <xacro:macro name="HDL-32E" params="*origin parent:=base_link name:=velodyne topic:=velodyne_points2 organize_cloud:=false hz:=15 lasers:=32 samples:=2187 collision_range:=0.3 min_range:=0.9 max_range:=130.0 noise:=0.008 min_angle:=-${M_PI} max_angle:=${M_PI} gpu:=false">
+  <xacro:macro name="HDL-32E" params="*origin parent:=base_link name:=velodyne topic:=velodyne_points2 organize_cloud:=false hz:=13 lasers:=32 samples:=2187 collision_range:=0.3 min_range:=0.9 max_range:=130.0 noise:=0.008 min_angle:=-${M_PI} max_angle:=${M_PI} gpu:=false">
     <joint name="${name}_base_mount_joint" type="fixed">
       <xacro:insert_block name="origin" />

File: src/genshin_simulation/urdf/VLP-16.xacro (robot description, xacro)
@@ -2,5 +2,5 @@
 <robot xmlns:xacro="http://www.ros.org/wiki/xacro" name="VLP-16">
   <xacro:property name="M_PI" value="3.1415926535897931" />
-  <xacro:macro name="VLP-16" params="*origin parent:=base_link name:=velodyne topic:=velodyne_points organize_cloud:=false hz:=15 lasers:=16 samples:=1875 collision_range:=0.3 min_range:=0.9 max_range:=130.0 noise:=0.008 min_angle:=-${M_PI} max_angle:=${M_PI} gpu:=false">
+  <xacro:macro name="VLP-16" params="*origin parent:=base_link name:=velodyne topic:=velodyne_points organize_cloud:=false hz:=13 lasers:=16 samples:=1875 collision_range:=0.3 min_range:=0.9 max_range:=130.0 noise:=0.008 min_angle:=-${M_PI} max_angle:=${M_PI} gpu:=false">
     <joint name="${name}_base_mount_joint" type="fixed">
       <xacro:insert_block name="origin" />

File: src/genshin_simulation/urdf/my_camera_sensor.xacro (robot description, xacro)
@@ -4,5 +4,5 @@
       <!-- 类型设置为 camara -->
       <sensor type="camera" name="camera_sim">
-        <update_rate>80.0</update_rate> <!-- 更新频率 -->
+        <update_rate>280.0</update_rate> <!-- 更新频率 -->
         <!-- 摄像头基本信息设置 -->
         <camera name="head">

File: src/genshin_simulation/urdf/my_car_HDL32.xacro (robot description, xacro)
@@ -1,2 +1,3 @@
+<?xml version="1.0"?>
 <robot name="my_car" xmlns:xacro="http://wiki.ros.org/xacro">
     <xacro:arg name="gpu" default="false" />
@@ -5,7 +6,12 @@
     <xacro:property name="organize_cloud" value="$(arg organize_cloud)" />
     <xacro:include filename="4w_mecanum.xacro" />
-    <xacro:include filename="HDL-32E.xacro"/>
-    <xacro:HDL-32E parent="base_link" name="velodyne2" topic="velodyne_points2" organize_cloud="${organize_cloud}" hz="15" samples="220" gpu="${gpu}">
+    <!-- <xacro:include filename="HDL-32E.xacro"/>
+    <xacro:HDL-32E parent="base_link" name="velodyne2" topic="velodyne_points2" organize_cloud="${organize_cloud}" hz="13" samples="220" gpu="${gpu}">
       <origin xyz="0 0 0.6" rpy="0 0 0" />
+    </xacro:HDL-32E> -->
+    <!-- <xacro:include filename="$(find genshin_simulation)/urdf/HDL-32E.urdf.xacro"/> -->
+    <xacro:include filename="HDL-32E.urdf.xacro"/>
+    <xacro:HDL-32E parent="base_link" name="velodyne2" topic="/velodyne_points2" organize_cloud="${organize_cloud}" hz="12" samples="320" gpu="${gpu}">
+      <origin xyz="0 0 0.4" rpy="0 0 0" />
     </xacro:HDL-32E>
     <xacro:include filename="my_imu.xacro" />
@@ -13,6 +19,3 @@
     <!-- <xacro:include filename="my_camera.xacro" />  -->
     <!-- <xacro:include filename="my_camera_sensor.xacro" /> -->
-    <!-- 二维雷达仿真，没必要注掉了 -->
-    <!-- <xacro:include filename="my_lidar.xacro" />
-    <xacro:include filename="my_lidar_sensor.xacro" /> -->
 </robot>

File: src/genshin_simulation/urdf/my_car_VLP16.xacro (robot description, xacro)
@@ -5,14 +5,11 @@
     <xacro:property name="organize_cloud" value="$(arg organize_cloud)" />
     <xacro:include filename="4w_mecanum.xacro" />
-    <xacro:include filename="VLP-16.xacro"/>
-    <xacro:VLP-16 parent="base_link" name="velodyne" topic="velodyne_points" organize_cloud="${organize_cloud}" hz="15" samples="440" gpu="${gpu}">
+    <xacro:include filename="VLP-16.urdf.xacro"/>
+    <xacro:VLP-16 parent="base_link" name="velodyne" topic="/velodyne_points" organize_cloud="${organize_cloud}" hz="12" samples="440" gpu="${gpu}">
       <origin xyz="0 0 0.4" rpy="0 0 0" />
     </xacro:VLP-16>
     <xacro:include filename="my_imu.xacro" />
     <!-- 摄像头仿真，没必要可以注掉 -->
-    <xacro:include filename="my_camera.xacro" />
-    <xacro:include filename="my_camera_sensor.xacro" />
-    <!-- 二维雷达仿真，没必要注掉了 -->
-    <!-- <xacro:include filename="my_lidar.xacro" />
-    <xacro:include filename="my_lidar_sensor.xacro" /> -->
+    <!-- <xacro:include filename="my_camera.xacro" />
+    <xacro:include filename="my_camera_sensor.xacro" /> -->
 </robot>

File: src/genshin_simulation/urdf/my_imu.xacro (robot description, xacro)
@@ -5,8 +5,4 @@
     <xacro:property name="imu_size" value="0.005" />
     <xacro:property name="imu_m" value="0.01" /> <!-- imu质量 -->
-    <plugin
-            filename="gz-sim-imu-system"
-            name="gz::sim::systems::Imu">
-        </plugin>
     <xacro:macro name="Box_inertial_matrix" params="m l w h">
         <inertial>
@@ -69,5 +65,5 @@
           </plugin>
           <always_on>true</always_on>
-          <update_rate>100</update_rate>
+          <update_rate>200</update_rate>
           <visualize>true</visualize>
           <imu>
